Commit message: Restructure final challenge package

File: urdf/puzzlebot.urdf (robot description, URDF)
Before this commit: robot puzzlebot, 5 links, 4 joints
Links:
- added link lidar_link, mass 0.05; collision cylinder length=0.035 radius=0.035; visual cylinder length=0.035 radius=0.035
Joints:
- added joint lidar_joint: type fixed, parent base_link, child lidar_link, origin xyz=0.06 0.0 0.12 rpy=0.0 0.0 0.0

Commit message: Add RPLidar mesh to robot URDF

File: urdf/puzzlebot.urdf (robot description, URDF)
Before this commit: robot puzzlebot, 6 links, 5 joints
Links:
- removed link lidar_link
- added link laser_frame, mass 0.00001; collision box size=0.005 0.005 0.005; visual box size=0.005 0.005 0.005
- added link lidar_base_link, mass 0.1755; collision box size=0.08 0.07 0.05; visual mesh filename=package://puzzlebot_sim2/meshes/RPLidar.stl scale=1 1 1
Joints:
- added joint lidar_base_joint: type fixed, parent base_link, child lidar_base_link, origin xyz=0.0425 0.0 0.070 rpy=0.0 0.0 0.0
- joint lidar_joint: child lidar_link -> laser_frame; origin xyz=0.06 0.0 0.12 rpy=0.0 0.0 0.0 -> xyz=0.0 0.0 0.035 rpy=0.0 0.0 0.0; parent base_link -> lidar_base_link

Commit message: added arucos

File: urdf/puzzlebot.urdf (robot description, URDF)
Before this commit: robot puzzlebot, 7 links, 6 joints
Links:
- added link camera_link, mass 0.01; collision box size=0.04 0.04 0.04; visual box size=0.04 0.04 0.04
Joints:
- added joint camera_joint: type fixed, parent base_link, child camera_link, origin xyz=0.10 0.0 0.10 rpy=0 0 0

Commit message: changes to git

File: urdf/puzzlebot.urdf (robot description, URDF)
Before this commit: robot puzzlebot, 8 links, 7 joints
Links:
- link camera_link: geometry collision box size=0.04 0.04 0.04; visual mesh filename=package://puzzlebot_sim2/meshes/Laser_Camera_Bracket.stl scale=1 1 1
