Commit message: npi1

File: urdf/mcr2_control/gazebo_control.xacro (robot description, xacro)
@@ -9,7 +9,7 @@
             <wheel_separation>0.19</wheel_separation>
             <wheel_radius>0.05</wheel_radius>
-            <topic>${prefix}cmd_vel</topic>
+            <topic>/${prefix}cmd_vel</topic>
             <tf_topic>diff_drive/tf</tf_topic>
-            <odom_topic>${prefix}odom</odom_topic>
+            <odom_topic>/${prefix}gz_odom</odom_topic>
             <frame_id>${prefix}odom</frame_id>
             <child_frame_id>${prefix}base_footprint</child_frame_id>
@@ -18,5 +18,5 @@
         </plugin>
         <plugin filename="gz-sim-joint-state-publisher-system" name="gz::sim::systems::JointStatePublisher">
-            <topic>${prefix}joint_states</topic>
+            <topic>/${prefix}joint_states</topic>
             <update_rate>50</update_rate>
             <joint_name>${prefix}wheel_right_joint</joint_name>
@@ -27,5 +27,5 @@
         <robot_base_frame>${prefix}base_footprint</robot_base_frame>
         <odom_publish_frequency>50</odom_publish_frequency>
-        <odom_topic>${prefix}ground_truth</odom_topic>
+        <odom_topic>/${prefix}ground_truth</odom_topic>
         <tf_topic>tf</tf_topic>
         <dimensions>2</dimensions>

File: urdf/mcr2_robots/hacker_ed/parameters_hacker_ed.xacro (robot description, xacro)
@@ -132,6 +132,6 @@
             <xacro:property name="wheel_pos_w" value="0.0"/>
     <!--Meshes -->
-        <xacro:property name="mesh_puzzlebot_chassis"  value="$(find puzzlebot_sim2)/meshes/bases/Puzzlebot_Hacker_Editon_Base.stl" />
-        <xacro:property name="mesh_puzzlebot_wheel"  value="$(find puzzlebot_sim2)/meshes/wheels/Puzzlebot_Wheel.stl" />
-        <xacro:property name="mesh_puzzlebot_caster"  value="$(find puzzlebot_sim2)/meshes/wheels/Puzzlebot_Caster_Wheel.stl" />
+        <xacro:property name="mesh_puzzlebot_chassis"  value="$(find final_challenge)/meshes/bases/Puzzlebot_Hacker_Editon_Base.stl" />
+        <xacro:property name="mesh_puzzlebot_wheel"  value="$(find final_challenge)/meshes/wheels/Puzzlebot_Wheel.stl" />
+        <xacro:property name="mesh_puzzlebot_caster"  value="$(find final_challenge)/meshes/wheels/Puzzlebot_Caster_Wheel.stl" />
 </robot>

File: urdf/mcr2_robots/jetson_ed/parameters_jetson_ed.xacro (robot description, xacro)
@@ -165,7 +165,7 @@
             <xacro:property name="jetson_pos_w" value="0.0"/>
     <!--Meshes -->
-        <xacro:property name="mesh_puzzlebot_chassis"  value="$(find puzzlebot_sim2)/meshes/bases/Puzzlebot_Hacker_Editon_Base.stl" />
-        <xacro:property name="mesh_puzzlebot_wheel"  value="$(find puzzlebot_sim2)/meshes/wheels/Puzzlebot_Wheel.stl" />
-        <xacro:property name="mesh_puzzlebot_caster"  value="$(find puzzlebot_sim2)/meshes/wheels/Puzzlebot_Caster_Wheel.stl" />
-        <xacro:property name="mesh_puzzlebot_jetson"  value="$(find puzzlebot_sim2)/meshes/misc/NVIDIA_Jetson.stl" />
+        <xacro:property name="mesh_puzzlebot_chassis"  value="$(find final_challenge)/meshes/bases/Puzzlebot_Hacker_Editon_Base.stl" />
+        <xacro:property name="mesh_puzzlebot_wheel"  value="$(find final_challenge)/meshes/wheels/Puzzlebot_Wheel.stl" />
+        <xacro:property name="mesh_puzzlebot_caster"  value="$(find final_challenge)/meshes/wheels/Puzzlebot_Caster_Wheel.stl" />
+        <xacro:property name="mesh_puzzlebot_jetson"  value="$(find final_challenge)/meshes/misc/NVIDIA_Jetson.stl" />
 </robot>

File: urdf/mcr2_robots/jetson_lidar_ed/parameters_jetson_lidar_ed.xacro (robot description, xacro)
@@ -165,7 +165,7 @@
             <xacro:property name="jetson_pos_w" value="0.0"/>
     <!--Meshes -->
-        <xacro:property name="mesh_puzzlebot_chassis"  value="$(find puzzlebot_sim2)/meshes/bases/Puzzlebot_Jetson_Lidar_Edition_Base.stl" />
-        <xacro:property name="mesh_puzzlebot_wheel"  value="$(find puzzlebot_sim2)/meshes/wheels/Puzzlebot_Wheel.stl" />
-        <xacro:property name="mesh_puzzlebot_caster"  value="$(find puzzlebot_sim2)/meshes/wheels/Puzzlebot_Caster_Wheel.stl" />
-        <xacro:property name="mesh_puzzlebot_jetson"  value="$(find puzzlebot_sim2)/meshes/misc/NVIDIA_Jetson.stl" />
+        <xacro:property name="mesh_puzzlebot_chassis"  value="$(find final_challenge)/meshes/bases/Puzzlebot_Jetson_Lidar_Edition_Base.stl" />
+        <xacro:property name="mesh_puzzlebot_wheel"  value="$(find final_challenge)/meshes/wheels/Puzzlebot_Wheel.stl" />
+        <xacro:property name="mesh_puzzlebot_caster"  value="$(find final_challenge)/meshes/wheels/Puzzlebot_Caster_Wheel.stl" />
+        <xacro:property name="mesh_puzzlebot_jetson"  value="$(find final_challenge)/meshes/misc/NVIDIA_Jetson.stl" />
 </robot>

File: urdf/mcr2_robots/puzzlebot_hacker_ed.xacro (robot description, xacro)
@@ -3,10 +3,10 @@
 <xacro:arg name="prefix" default=""/>
 <!-- files for gazebo costumization -->
-<xacro:include filename="$(find puzzlebot_sim2)/urdf/mcr2_mechanical/puzzlebot_hacker_base.urdf.xacro"/>
-<xacro:include filename="$(find puzzlebot_sim2)/urdf/mcr2_robots/hacker_ed/parameters_hacker_ed.xacro" />
-<xacro:include filename="$(find puzzlebot_sim2)/urdf/mcr2_misc/materials.xacro" />
-<xacro:include filename="$(find puzzlebot_sim2)/urdf/mcr2_misc/macros.xacro" />
-<xacro:include filename="$(find puzzlebot_sim2)/urdf/mcr2_sensors/laser_camera_bracket.xacro" />
-<xacro:include filename="$(find puzzlebot_sim2)/urdf/mcr2_control/gazebo_control.xacro" />
+<xacro:include filename="$(find final_challenge)/urdf/mcr2_mechanical/puzzlebot_hacker_base.urdf.xacro"/>
+<xacro:include filename="$(find final_challenge)/urdf/mcr2_robots/hacker_ed/parameters_hacker_ed.xacro" />
+<xacro:include filename="$(find final_challenge)/urdf/mcr2_misc/materials.xacro" />
+<xacro:include filename="$(find final_challenge)/urdf/mcr2_misc/macros.xacro" />
+<xacro:include filename="$(find final_challenge)/urdf/mcr2_sensors/laser_camera_bracket.xacro" />
+<xacro:include filename="$(find final_challenge)/urdf/mcr2_control/gazebo_control.xacro" />
 <!--LINKS-->
 <xacro:puzzlebot_hacker_ed_base prefix="$(arg prefix)" />

File: urdf/mcr2_robots/puzzlebot_jetson_ed.xacro (robot description, xacro)
@@ -3,10 +3,10 @@
 <xacro:arg name="prefix" default=""/>
 <!-- files for gazebo costumization -->
-<xacro:include filename="$(find puzzlebot_sim2)/urdf/mcr2_mechanical/puzzlebot_jetson_base.urdf.xacro"/>
-<xacro:include filename="$(find puzzlebot_sim2)/urdf/mcr2_robots/jetson_ed/parameters_jetson_ed.xacro" />
-<xacro:include filename="$(find puzzlebot_sim2)/urdf/mcr2_misc/materials.xacro" />
-<xacro:include filename="$(find puzzlebot_sim2)/urdf/mcr2_misc/macros.xacro" />
-<xacro:include filename="$(find puzzlebot_sim2)/urdf/mcr2_sensors/laser_camera_bracket.xacro" />
-<xacro:include filename="$(find puzzlebot_sim2)/urdf/mcr2_control/gazebo_control.xacro" />
+<xacro:include filename="$(find final_challenge)/urdf/mcr2_mechanical/puzzlebot_jetson_base.urdf.xacro"/>
+<xacro:include filename="$(find final_challenge)/urdf/mcr2_robots/jetson_ed/parameters_jetson_ed.xacro" />
+<xacro:include filename="$(find final_challenge)/urdf/mcr2_misc/materials.xacro" />
+<xacro:include filename="$(find final_challenge)/urdf/mcr2_misc/macros.xacro" />
+<xacro:include filename="$(find final_challenge)/urdf/mcr2_sensors/laser_camera_bracket.xacro" />
+<xacro:include filename="$(find final_challenge)/urdf/mcr2_control/gazebo_control.xacro" />
 <!--LINKS-->
 <xacro:puzzlebot_jetson_ed_base prefix="$(arg prefix)" />

File: urdf/mcr2_robots/puzzlebot_jetson_lidar_ed.xacro (robot description, xacro)
@@ -3,11 +3,11 @@
 <xacro:arg name="prefix" default=""/>
 <!-- files for gazebo costumization -->
-<xacro:include filename="$(find puzzlebot_sim2)/urdf/mcr2_mechanical/puzzlebot_jetson_lidar_base.urdf.xacro"/>
-<xacro:include filename="$(find puzzlebot_sim2)/urdf/mcr2_robots/jetson_lidar_ed/parameters_jetson_lidar_ed.xacro" />
-<xacro:include filename="$(find puzzlebot_sim2)/urdf/mcr2_misc/materials.xacro" />
-<xacro:include filename="$(find puzzlebot_sim2)/urdf/mcr2_misc/macros.xacro" />
-<xacro:include filename="$(find puzzlebot_sim2)/urdf/mcr2_sensors/laser_camera_bracket.xacro" />
-<xacro:include filename="$(find puzzlebot_sim2)/urdf/mcr2_sensors/lidar.xacro" />
-<xacro:include filename="$(find puzzlebot_sim2)/urdf/mcr2_control/gazebo_control.xacro" />
+<xacro:include filename="$(find final_challenge)/urdf/mcr2_mechanical/puzzlebot_jetson_lidar_base.urdf.xacro"/>
+<xacro:include filename="$(find final_challenge)/urdf/mcr2_robots/jetson_lidar_ed/parameters_jetson_lidar_ed.xacro" />
+<xacro:include filename="$(find final_challenge)/urdf/mcr2_misc/materials.xacro" />
+<xacro:include filename="$(find final_challenge)/urdf/mcr2_misc/macros.xacro" />
+<xacro:include filename="$(find final_challenge)/urdf/mcr2_sensors/laser_camera_bracket.xacro" />
+<xacro:include filename="$(find final_challenge)/urdf/mcr2_sensors/lidar.xacro" />
+<xacro:include filename="$(find final_challenge)/urdf/mcr2_control/gazebo_control.xacro" />
 <!--LINKS-->
 <xacro:puzzlebot_jetson_lidar_ed_base prefix="$(arg prefix)" />

File: urdf/mcr2_sensors/laser_camera_bracket.xacro (robot description, xacro)
@@ -6,5 +6,5 @@
     camera_name:='cam_1'
     parent:='base_link'
-    mesh_file:='file://$(find puzzlebot_sim2)/meshes/sensors/Laser_Camera_Bracket.stl'
+    mesh_file:='file://$(find final_challenge)/meshes/sensors/Laser_Camera_Bracket.stl'
     camera_base_mass:='0.035'
     camera_base_length:='0.046'

File: urdf/mcr2_sensors/lidar.xacro (robot description, xacro)
@@ -6,5 +6,5 @@
     frame_name:='laser_frame'
     parent:='base_link'
-    mesh_file:='file://$(find puzzlebot_sim2)/meshes/sensors/RPLidar.stl'
+    mesh_file:='file://$(find final_challenge)/meshes/sensors/RPLidar.stl'
     lidar_base_mass:='0.1755'
     lidar_base_length:='0.08'
@@ -110,5 +110,5 @@
     <gazebo reference="${prefix}laser_frame">
         <sensor name="${prefix}lidar_sensor" type="gpu_lidar">
-            <topic>${prefix}${topic_name}</topic>
+            <topic>/${prefix}${topic_name}</topic>
             <gz_frame_id>${prefix}laser_frame</gz_frame_id>
             <pose> 0 0 0 0 0 0 </pose>
